Commit message: feat(base): improve mecanum odometry and serial bridge

File: src/robot_description/urdf/sensors.xacro (robot description, xacro)
@@ -46,3 +46,21 @@
     <origin xyz="0 -0.030 0" rpy="0 0 0"/>
   </joint>
+  <link name="camera_left_optical_frame"/>
+<joint name="camera_left_optical_joint"
+       type="fixed">
+  <parent link="camera_left_link"/>
+  <child link="camera_left_optical_frame"/>
+  <origin
+    xyz="0 0 0"
+    rpy="-1.5708 0 -1.5708"/>
+</joint>
+<link name="camera_right_optical_frame"/>
+<joint name="camera_right_optical_joint"
+       type="fixed">
+  <parent link="camera_right_link"/>
+  <child link="camera_right_optical_frame"/>
+  <origin
+    xyz="0 0 0"
+    rpy="-1.5708 0 -1.5708"/>
+</joint>
 </robot>
